File: PFD_HMC439QS16G.sch (KiCad schematic (older format))
At the start: 68 parts, among them J1 REF, J2 IN, J3 Error_Out, J4 C64AC, J5 Fast_Out, U1 HMC439QS16G, U2 LT3045EMSE, U3 LT3094EMSE, U4 ADA4896-2ARMZ, U5 ADA4896-2ARMZ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

Commit message: Add LM7908 and TVS diodes for line protection
Parts:
- added C2, C28: 100u, Capacitor_THT:CP_Radial_D5.0mm_P2.50mm, symbol Device:CP_Small
- added C25, C27: 100n, Capacitor_SMD:C_0603_1608Metric, symbol Device:C_Small
- added D1, D2: SMB, Diode_SMD:D_SMB, symbol Device:D_TVS
- added U6: LM7908_TO220, Package_TO_SOT_THT:TO-220-3_Horizontal_TabDown, symbol Regulator_Linear:LM7908_TO220
- U7: value L7809 -> LM7808; symbol Regulator_Linear:L7809 -> Regulator_Linear:LM7808_TO220
Connections:
- net +15V: now also D1.1 (A1)
- net GND: now also C2.1, C25.1, C27.1, C28.1, D1.2 (A2), D2.2 (A2), U6.1 (GND)
- net IN: now also C27.2, C28.2, U6.3 (VO); no longer J4.A31 (31A), J4.A32 (32A), J4.C31 (31C), J4.C32 (32C)
- new net -15V: C2.2, C25.2, D2.1 (A1), J4.A31 (31A), J4.A32 (32A), J4.C31 (31C), J4.C32 (32C), U6.2 (VI)
Other:
- moved on the sheet: C29, C30, C31, C32, U7
