File: PFD_HMC439QS16G.kicad_sch (KiCad schematic)
At the start: 63 parts, among them J1 REF, J2 IN, J3 Error_Out, J4 C64AC, U1 HMC439QS16G, U2 LT3045EMSE, U3 LT3094EMSE, U4 ADA4896-2ARMZ, U6 HMC365S8G, U7 L7808

Commit message: Update BOM / fix some fottprints
Parts:
- C1, C2, C25: MFN (none) -> TDK; PN (none) -> CGJ3E2C0G2A101J080AA
- C16: value 140p -> 150p
- C26: footprint Capacitor_SMD:C_0603_1608Metric_Pad1.08x0.95mm_HandSolder -> Capacitor_SMD:C_0603_1608Metric; MFN (none) -> TDK; PN (none) -> CGJ3E2C0G2A101J080AA
- C7, C8: value 0.47u -> 100n; MFN (none) -> Murata-Electronics; PN (none) -> GRM3195C2A104JA01D
- D1, D2: MFN (none) -> Bourns; PN (none) -> SMBJ40CA-QH
- JP1, JP2, LOGO1, LOGO2, LOGO3: Config (none) -> DNF
- R10, R11: value 380 -> 390; MFN (none) -> Yageo; PN (none) -> RC0603FR-13390RL
- R12, R13, R3, R4, R5, R8, R9: MFN (none) -> Yageo; PN (none) -> RC0603FR-13200RL
- R14: MFN (none) -> Yageo; PN (none) -> RC0603FR-13100RL
- R6, R7: MFN (none) -> Yageo; PN (none) -> AC0603FR-0720RL
- U1: MFN (none) -> Analog Devices
- U2: MFN Linear Technology -> Analog Devices; MFP LT3045EMSE -> (none); PN (none) -> LT3045EMSE#PBF
- U3: MFN Linear Technology -> Analog Devices; MFP LT3094EMSE -> (none); PN (none) -> LT3094EMSE#PBF
- U4: MFN (none) -> Analog Devices; PN (none) -> ADA4896-2ARMZ
- U6: MFN (none) -> Analog Devices; PN (none) -> HMC365S8GETR

Commit message: Updated BOM with new parts
Parts:
- C10, C19, C27, C5, C6: MFN (none) -> KEMET; PN (none) -> C0603X102K4RACAUTO
- C11, C12, C3, C4: MFN (none) -> TDK; PN (none) -> C3225X7R2A106K250AC
- C13, C14, C20: MFN (none) -> Vishay / Vitramon; PN (none) -> VJ0603A150JXBAC
- C15: MFN (none) -> Vishay / Vitramon; PN (none) -> VJ0603A561JXAAC
- C16: MFN (none) -> Vishay / Vitramon; PN (none) -> VJ0603A151JXBAC
- C17, C18, C28, C30, C31, C9: MFN (none) -> KEMET; PN (none) -> C0603C104K5RAC3121
- C21, C29, C32: MFN (none) -> Panasonic; PN (none) -> ECA-1AM101I
- J1, J2: MFN (none) -> Linx Technologies; PN (none) -> CONREVSMA006.062-G
- J3: MFN (none) -> Linx Technologies; PN (none) -> CONBNC002
- J4: MFN (none) -> HARTING; PN (none) -> 09221326921222
- R1, R2: MFN (none) -> Panasonic; PN (none) -> ERJ-UP3F4992V
- R15: MFN (none) -> Vishay / Dale; PN (none) -> CRCW121049R9FKEA
- R20: MFN (none) -> Panasonic; PN (none) -> ERJ-UP3F49R9V
- U1, U6: Config (none) -> DNF
- U7: MFN (none) -> STMicroelectronics; PN (none) -> L7808ABV-DG

Commit message: Update BOM
Parts:
- J4: MFN HARTING -> Harting
- U1: PN (none) -> HMC439QS16GE
Changed lines of the file:
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@@
+      (effects (font (size 1.27 1.27)) hide)
+    )
+    (property "PN" "HMC439QS16GE" (id 6) (at 77.47 124.46 0)
       (effects (font (size 1.27 1.27)) hide)
     )
@@
       (effects (font (size 1.27 1.27)) hide)
     )
-    (property "MFN" "HARTING " (id 4) (at 20.32 147.32 0)
-      (effects (font (size 1.27 1.27)) hide)
-    )
+    (property "MFN" "Harting" (id 4) (at 20.32 147.32 0)
+      (effects (font (size 1.27 1.27)) hide)
+    )
