File: phase-frequency_detector.kicad_sch (KiCad schematic)
At the start: 63 parts, among them J1 REF, J2 IN, J3 Error_Out, J4 C64AC, U1 HMC439QS16G, U2 LT3045EMSE, U3 LT3094EMSE, U4 ADA4896-2ARMZ, U6 HMC365S8G, U7 L7808

Commit message: Add comments and fix custom footprint lib.
Other:
- note added: "Close JP1 and JP2, if the divider (U6) is not used."
- note added: "Input frequency range With divider (U6): 0.5 to 5.2 GHz Without divider: 0.01 to 1.3 GHz"
Changed lines of the file:
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@@
     (stroke (width 0) (type default) (color 0 0 0 0))
+  )
+  (text "Input frequency range\nWith divider (U6): 0.5 to 5.2 GHz\nWithout divider: 0.01 to 1.3 GHz\n"
+    (at 26.67 29.845 0)
+    (effects (font (size 1.524 1.524)) (justify left bottom))
+  )
+  (text "Close JP1 and JP2,\nif the divider (U6)\nis not used.\n"
+    (at 150.495 21.59 0)
+    (effects (font (size 1.524 1.524)) (justify left bottom))
   )
   (global_label "+8V" (shape output) (at 215.9 139.7 0) (fields_autoplaced)

Commit message: Remove solder paste from DNF footprints.
Parts:
- U1: footprint footprints:QSOP-16_3.9x4.9mm_P0.635mm_EP_2.3mmx1.75mm -> footprints:QSOP-16_3.9x4.9mm_P0.635mm_EP_2.3mmx1.75mm_DNF
- U6: footprint Package_SO:SOIC-8-1EP_3.9x4.9mm_P1.27mm_EP2.41x3.81mm -> footprints:SOIC-8-1EP_3.9x4.9mm_P1.27mm_EP2.41x3.81mm_DNF
Other:
- title: HMC439 Phase-Frequency Detector -> Phase-Frequency Detector
Changed lines of the file:
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@@
   (paper "A4")
   (title_block
-    (title "HMC439 Phase-Frequency Detector")
-    (date "2022-01-25")
-    (rev "1.4")
+    (title "Phase-Frequency Detector")
+    (date "2023-03-22")
+    (rev "1.4.1")
     (company "Atoms-Photons-Quanta, IAP, TU Darmstadt")
     (comment 1 "Tilman Preuschoff")
@@
       (effects (font (size 1.524 1.524)))
     )
-    (property "Footprint" "footprints:QSOP-16_3.9x4.9mm_P0.635mm_EP_2.3mmx1.75mm" (id 2) (at 77.47 124.46 0)
+    (property "Footprint" "footprints:QSOP-16_3.9x4.9mm_P0.635mm_EP_2.3mmx1.75mm_DNF" (id 2) (at 77.47 124.46 0)
       (effects (font (size 1.524 1.524)) hide)
     )
@@
       (effects (font (size 1.524 1.524)))
     )
-    (property "Footprint" "Package_SO:SOIC-8-1EP_3.9x4.9mm_P1.27mm_EP2.41x3.81mm" (id 2) (at 114.3 53.34 0)
+    (property "Footprint" "footprints:SOIC-8-1EP_3.9x4.9mm_P1.27mm_EP2.41x3.81mm_DNF" (id 2) (at 114.3 53.34 0)
       (effects (font (size 1.524 1.524)) hide)
     )
@@
     )
     (path "/00000000-0000-0000-0000-00005c6b12de"
-      (reference "U1") (unit 1) (value "HMC439QS16G") (footprint "footprints:QSOP-16_3.9x4.9mm_P0.635mm_EP_2.3mmx1.75mm")
+      (reference "U1") (unit 1) (value "HMC439QS16G") (footprint "footprints:QSOP-16_3.9x4.9mm_P0.635mm_EP_2.3mmx1.75mm_DNF")
     )
     (path "/00000000-0000-0000-0000-00005c669751"
@@
     )
     (path "/00000000-0000-0000-0000-00006058f7be"
-      (reference "U6") (unit 1) (value "HMC365S8G") (footprint "Package_SO:SOIC-8-1EP_3.9x4.9mm_P1.27mm_EP2.41x3.81mm")
+      (reference "U6") (unit 1) (value "HMC365S8G") (footprint "footprints:SOIC-8-1EP_3.9x4.9mm_P1.27mm_EP2.41x3.81mm_DNF")
     )
     (path "/00000000-0000-0000-0000-00006072aebc"

Commit message: Update gerber files
Parts:
- J1, J2: MFN Linx Technologies -> Amphenol; PN CONREVSMA006.062-G -> 132289
Changed lines of the file:
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@@
       (effects (font (size 1.27 1.27)) hide)
     )
-    (property "MFN" "Linx Technologies " (id 4) (at 33.02 88.9 0)
-      (effects (font (size 1.27 1.27)) hide)
-    )
-    (property "PN" "CONREVSMA006.062-G " (id 5) (at 33.02 88.9 0)
+    (property "MFN" "Amphenol" (id 4) (at 33.02 88.9 0)
+      (effects (font (size 1.27 1.27)) hide)
+    )
+    (property "PN" "132289" (id 5) (at 33.02 88.9 0)
       (effects (font (size 1.27 1.27)) hide)
     )
@@
       (effects (font (size 1.27 1.27)) hide)
     )
-    (property "MFN" "Linx Technologies " (id 4) (at 72.39 27.94 0)
-      (effects (font (size 1.27 1.27)) hide)
-    )
-    (property "PN" "CONREVSMA006.062-G " (id 5) (at 72.39 27.94 0)
-      (effects (font (size 1.27 1.27)) hide)
-    )
+    (property "MFN" "Amphenol" (id 4) (at 72.39 27.94 0)
+      (effects (font (size 1.27 1.27)) hide)
+    )
+    (property "PN" "132289" (id 5) (at 72.39 27.94 0)
+      (effects (font (size 1.27 1.27)) hide)
+    )

Commit message: Correct PN for Harting and BNC connectors
Parts:
- J4: PN 09221326921222 -> 9031646921
Changed lines of the file:
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@@
       (effects (font (size 1.27 1.27)) hide)
     )
-    (property "PN" "09221326921222 " (id 5) (at 20.32 147.32 0)
+    (property "PN" "9031646921" (id 5) (at 20.32 147.32 0)
       (effects (font (size 1.27 1.27)) hide)
     )
@@
     )
     (path "/00000000-0000-0000-0000-0000620090fe/00000000-0000-0000-0000-000061fb0f2a"
-      (reference "U8") (unit 1) (value "ADG1413") (footprint "Package_SO:TSSOP-16_4.4x5mm_P0.65mm")
+      (reference "U8") (unit 1) (value "ADG1613") (footprint "Package_SO:TSSOP-16_4.4x5mm_P0.65mm")
     )
     (path "/00000000-0000-0000-0000-0000620090fe/00000000-0000-0000-0000-000061eb46ba"
