File: PD_regulator.kicad_sch (KiCad schematic)
At the start: 26 parts, among them J5 Switch, J6 Fast_Out, U5 ADA4896-2ARMZ, U8 ADG1613, U9 LTC6228xS8

Commit message: Updated to KiCad 7 Added CI pipeline Fixed trailing whitespaces of MFN and PN labels Fixed ERC/DRC errors
Parts:
- C22, C23, C33, C34, C36, C37, C39: PN C0603C104K5RAC3121 -> C0603C104K5RAC3121
- C24: MFN Vishay / Vitramon -> Vishay / Vitramon; PN VJ0603A150JXBAC -> VJ0603A150JXBAC
- C35: PN C0603X102K4RACAUTO -> C0603X102K4RACAUTO
- J6: MFN Linx Technologies -> Linx Technologies
- R24: MFN ROHM Semiconductor -> ROHM Semiconductor
- R26: MFN Vishay / Dale -> Vishay / Dale; PN CRCW121049R9FKEA -> CRCW121049R9FKEA
- RV1: MFN Vishay / Spectrol -> Vishay / Spectrol; PN M43P501KB40 -> M43P501KB40
Other:
- company: Atoms-Photons-Quanta, IAP, TU Darmstadt -> Atoms-Photons-Quanta, Institut für Angewandte Physik, TU Darmstadt
